File: pcb/audio.kicad_sch (KiCad schematic)
At the start: 23 parts, among them J301 SPK2, J302 SPK1, U301 TAS5805M

Commit message: schematic and tweaks
Parts:
- C301, C302: footprint (none) -> Capacitor_SMD:C_0402_1005Metric; LCSC (none) -> C52923
- C303, C309, C314: footprint (none) -> Capacitor_SMD:C_0402_1005Metric; LCSC (none) -> C307331
- C304: value 4.7u -> 10u; footprint (none) -> Capacitor_SMD:C_0603_1608Metric; LCSC (none) -> C96446
- C305, C306, C307, C308: footprint (none) -> Capacitor_SMD:C_0805_2012Metric; LCSC (none) -> C5378
- C310, C315: footprint (none) -> Capacitor_SMD:C_0805_2012Metric; LCSC (none) -> C3882769; Notes (none) -> JB
- C311, C313: footprint (none) -> Capacitor_SMD:C_0805_2012Metric; LCSC (none) -> C107133
- C312: value 390u -> 330u; footprint (none) -> Capacitor_SMD:CP_Elec_10x10.5; LCSC (none) -> C88796; Notes (none) -> 35V
- C316: value 390u -> 330u; footprint (none) -> Capacitor_SMD:CP_Elec_10x10.5; LCSC (none) -> C88796
- J301, J302: LCSC (none) -> C3095360
- L301, L302: value 10u -> 10uH
Connections:
- net PVDD renamed +20V
