File: pcb/power.kicad_sch (KiCad schematic)
At the start: 19 parts, among them J401 ADC-055B-9, J402 USBC, J403 ADC-055B-9, U401 TPS62932

Commit message: schematic and tweaks
Parts:
- added J404: 20V, Connector_PinSocket_2.54mm:PinSocket_1x02_P2.54mm_Horizontal, symbol Connector:Conn_01x02_Socket
- added J405: 20v, Connector_PinHeader_2.54mm:PinHeader_1x02_P2.54mm_Horizontal, symbol Connector:Conn_01x02_Pin
- C401: value 33n -> 100n; footprint (none) -> Capacitor_SMD:C_0402_1005Metric; LCSC (none) -> C307331; Notes (none) -> 18mS
- C402: footprint Capacitor_SMD:C_1206_3216Metric -> Capacitor_SMD:C_0805_2012Metric; LCSC C13585 -> C440198
- C403: footprint Capacitor_SMD:C_0603_1608Metric -> Capacitor_SMD:C_0402_1005Metric; LCSC C14663 -> C307331; Notes 50v -> 50v(ignore)
- C404: value 0.1u -> 100n; footprint Capacitor_SMD:C_0603_1608Metric -> Capacitor_SMD:C_0402_1005Metric; LCSC C14663 -> C307331
- C405, C407, C408: LCSC C19702 -> C96446
Connections:
- net +20V: now also J405.1 (Pin_1); no longer J401.1
- net GND: now also J404.2 (Pin_2), J405.2 (Pin_2)
- new net: J401.1, J404.1 (Pin_1)
Other:
- moved on the sheet: J401, J403
